File: EIBs/Hirose128-Expanded/DR_EIB-128_expandedv1.3.brd (EAGLE design)
At the start: 26.9 x 37.5 mm, 129 parts

Commit message: Updated Neuralynx breakout board before manufacturing
Connections:
- net N$100 renamed T24_2
- net N$102 renamed T24_3
- net N$104 renamed T24_4
- net N$106 renamed T25_1
- net N$108 renamed T25_2
- net N$110 renamed T25_3
- net N$112 renamed T25_4
- net N$114 renamed T26_1
- net N$116 renamed T26_2
- net N$118 renamed T26_3
- net N$120 renamed T26_4
- net N$121 renamed T12_1
- net N$122 renamed T11_4
- net N$123 renamed T12_2
- net N$124 renamed T11_3
- net N$125 renamed T12_3
- net N$126 renamed T11_2
- net N$127 renamed T12_4
- net N$128 renamed T11_1
- net N$33 renamed T5_4
- net N$35 renamed T5_3
- net N$37 renamed T5_2
- net N$39 renamed T5_1
- net N$41 renamed T4_4
- net N$43 renamed T4_3
- net N$45 renamed T4_2
- net N$47 renamed T4_1
- net N$49 renamed T3_4
- net N$51 renamed T3_3
- net N$53 renamed T3_2
- net N$55 renamed T3_1
- net N$57 renamed T2_1
- net N$59 renamed T2_2
- net N$61 renamed T2_3
- net N$63 renamed T2_4
- net N$65 renamed T9_1
- net N$66 renamed T10_4
- net N$67 renamed T9_2
- net N$68 renamed T10_3
- net N$69 renamed T9_3
- net N$70 renamed T10_2
- net N$71 renamed T9_4
- net N$72 renamed T10_1
- net N$73 renamed T8_4
- net N$74 renamed T21_1
- net N$75 renamed T8_3
- net N$76 renamed T21_2
- net N$77 renamed T8_2
- net N$78 renamed T21_3
- net N$79 renamed T8_1
- net N$80 renamed T21_4
- net N$81 renamed T7_4
- net N$82 renamed T22_1
- net N$83 renamed T7_3
- net N$84 renamed T22_2
- net N$85 renamed T7_2
- net N$86 renamed T22_3
- net N$87 renamed T7_1
- net N$88 renamed T22_4
- net N$89 renamed T6_4
- net N$90 renamed T23_1
- net N$91 renamed T6_3
- net N$92 renamed T23_2
- net N$93 renamed T6_2
- net N$94 renamed T23_3
- net N$95 renamed T6_1
- net N$96 renamed T23_4
- net N$98 renamed T24_1
