File: EIBs/Hirose128 Circle/DR_EIB-128_Circle_0_25MM.sch (EAGLE design)
At the start: 42 parts

Commit message: Three updates for Circular EIB: - Add library with the radial tetrode configuration (1.5 in diameter) in 0.3 mm and 0.25 mm tetrode holes - Update CircleEIB files with 0.3 mm tetrode hole specification (also update DRC with 0.3 mm minimum drill) - Add second CircleEIB files with 0.25 mm tetrode holes
Parts:
- 0, 1, 10, 11, 12, 13, 14, 15, 16, 17, 18, 19, 2, 20, 21, 22, 23, 24, 25, 26, 27, 28, 29, 3, 30, 31, 4, 5, 6, 7, 8, 9: value TETRODE_1.5IN_RADIUS0.3MM -> TETRODE_1.5IN_RADIUS0.25MM; device CactusPinInterfaces:TETRODE_1.5IN_RADIUS0.3MM -> CactusPinInterfaces:TETRODE_1.5IN_RADIUS0.25MM
Changed lines of the file:
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@@
 <part name="U$11" library="UsefulConnectors" deviceset="HIROSE-70PIN-HEADER" device="-SEQUENTIAL" value="HIROSE-70PIN-HEADER-SEQUENTIAL"/>
 <part name="GND2" library="supply1" library_urn="urn:adsk.eagle:library:371" deviceset="GND" device=""/>
-<part name="0" library="CactusPinInterfaces" deviceset="TETRODE_1.5IN_RADIUS" device="0.3MM"/>
-<part name="1" library="CactusPinInterfaces" deviceset="TETRODE_1.5IN_RADIUS" device="0.3MM"/>
-<part name="2" library="CactusPinInterfaces" deviceset="TETRODE_1.5IN_RADIUS" device="0.3MM"/>
-<part name="3" library="CactusPinInterfaces" deviceset="TETRODE_1.5IN_RADIUS" device="0.3MM"/>
-<part name="4" library="CactusPinInterfaces" deviceset="TETRODE_1.5IN_RADIUS" device="0.3MM"/>
-<part name="5" library="CactusPinInterfaces" deviceset="TETRODE_1.5IN_RADIUS" device="0.3MM"/>
-<part name="6" library="CactusPinInterfaces" deviceset="TETRODE_1.5IN_RADIUS" device="0.3MM"/>
-<part name="7" library="CactusPinInterfaces" deviceset="TETRODE_1.5IN_RADIUS" device="0.3MM"/>
-<part name="8" library="CactusPinInterfaces" deviceset="TETRODE_1.5IN_RADIUS" device="0.3MM"/>
-<part name="9" library="CactusPinInterfaces" deviceset="TETRODE_1.5IN_RADIUS" device="0.3MM"/>
-<part name="10" library="CactusPinInterfaces" deviceset="TETRODE_1.5IN_RADIUS" device="0.3MM"/>
-<part name="11" library="CactusPinInterfaces" deviceset="TETRODE_1.5IN_RADIUS" device="0.3MM"/>
-<part name="12" library="CactusPinInterfaces" deviceset="TETRODE_1.5IN_RADIUS" device="0.3MM"/>
-<part name="13" library="CactusPinInterfaces" deviceset="TETRODE_1.5IN_RADIUS" device="0.3MM"/>
-<part name="14" library="CactusPinInterfaces" deviceset="TETRODE_1.5IN_RADIUS" device="0.3MM"/>
-<part name="15" library="CactusPinInterfaces" deviceset="TETRODE_1.5IN_RADIUS" device="0.3MM"/>
-<part name="16" library="CactusPinInterfaces" deviceset="TETRODE_1.5IN_RADIUS" device="0.3MM"/>
-<part name="17" library="CactusPinInterfaces" deviceset="TETRODE_1.5IN_RADIUS" device="0.3MM"/>
-<part name="18" library="CactusPinInterfaces" deviceset="TETRODE_1.5IN_RADIUS" device="0.3MM"/>
-<part name="19" library="CactusPinInterfaces" deviceset="TETRODE_1.5IN_RADIUS" device="0.3MM"/>
-<part name="20" library="CactusPinInterfaces" deviceset="TETRODE_1.5IN_RADIUS" device="0.3MM"/>
-<part name="21" library="CactusPinInterfaces" deviceset="TETRODE_1.5IN_RADIUS" device="0.3MM"/>
-<part name="22" library="CactusPinInterfaces" deviceset="TETRODE_1.5IN_RADIUS" device="0.3MM"/>
-<part name="23" library="CactusPinInterfaces" deviceset="TETRODE_1.5IN_RADIUS" device="0.3MM"/>
-<part name="24" library="CactusPinInterfaces" deviceset="TETRODE_1.5IN_RADIUS" device="0.3MM"/>
-<part name="25" library="CactusPinInterfaces" deviceset="TETRODE_1.5IN_RADIUS" device="0.3MM"/>
-<part name="26" library="CactusPinInterfaces" deviceset="TETRODE_1.5IN_RADIUS" device="0.3MM"/>
-<part name="27" library="CactusPinInterfaces" deviceset="TETRODE_1.5IN_RADIUS" device="0.3MM"/>
-<part name="28" library="CactusPinInterfaces" deviceset="TETRODE_1.5IN_RADIUS" device="0.3MM"/>
-<part name="29" library="CactusPinInterfaces" deviceset="TETRODE_1.5IN_RADIUS" device="0.3MM"/>
-<part name="30" library="CactusPinInterfaces" deviceset="TETRODE_1.5IN_RADIUS" device="0.3MM"/>
-<part name="31" library="CactusPinInterfaces" deviceset="TETRODE_1.5IN_RADIUS" device="0.3MM"/>
+<part name="0" library="CactusPinInterfaces" deviceset="TETRODE_1.5IN_RADIUS" device="0.25MM" value="TETRODE_1.5IN_RADIUS0.25MM"/>
+<part name="1" library="CactusPinInterfaces" deviceset="TETRODE_1.5IN_RADIUS" device="0.25MM" value="TETRODE_1.5IN_RADIUS0.25MM"/>
+<part name="2" library="CactusPinInterfaces" deviceset="TETRODE_1.5IN_RADIUS" device="0.25MM" value="TETRODE_1.5IN_RADIUS0.25MM"/>
+<part name="3" library="CactusPinInterfaces" deviceset="TETRODE_1.5IN_RADIUS" device="0.25MM" value="TETRODE_1.5IN_RADIUS0.25MM"/>
+<part name="4" library="CactusPinInterfaces" deviceset="TETRODE_1.5IN_RADIUS" device="0.25MM" value="TETRODE_1.5IN_RADIUS0.25MM"/>
+<part name="5" library="CactusPinInterfaces" deviceset="TETRODE_1.5IN_RADIUS" device="0.25MM" value="TETRODE_1.5IN_RADIUS0.25MM"/>
+<part name="6" library="CactusPinInterfaces" deviceset="TETRODE_1.5IN_RADIUS" device="0.25MM" value="TETRODE_1.5IN_RADIUS0.25MM"/>
+<part name="7" library="CactusPinInterfaces" deviceset="TETRODE_1.5IN_RADIUS" device="0.25MM" value="TETRODE_1.5IN_RADIUS0.25MM"/>
+<part name="8" library="CactusPinInterfaces" deviceset="TETRODE_1.5IN_RADIUS" device="0.25MM" value="TETRODE_1.5IN_RADIUS0.25MM"/>
+<part name="9" library="CactusPinInterfaces" deviceset="TETRODE_1.5IN_RADIUS" device="0.25MM" value="TETRODE_1.5IN_RADIUS0.25MM"/>
+<part name="10" library="CactusPinInterfaces" deviceset="TETRODE_1.5IN_RADIUS" device="0.25MM" value="TETRODE_1.5IN_RADIUS0.25MM"/>
+<part name="11" library="CactusPinInterfaces" deviceset="TETRODE_1.5IN_RADIUS" device="0.25MM" value="TETRODE_1.5IN_RADIUS0.25MM"/>
+<part name="12" library="CactusPinInterfaces" deviceset="TETRODE_1.5IN_RADIUS" device="0.25MM" value="TETRODE_1.5IN_RADIUS0.25MM"/>
+<part name="13" library="CactusPinInterfaces" deviceset="TETRODE_1.5IN_RADIUS" device="0.25MM" value="TETRODE_1.5IN_RADIUS0.25MM"/>
+<part name="14" library="CactusPinInterfaces" deviceset="TETRODE_1.5IN_RADIUS" device="0.25MM" value="TETRODE_1.5IN_RADIUS0.25MM"/>
+<part name="15" library="CactusPinInterfaces" deviceset="TETRODE_1.5IN_RADIUS" device="0.25MM" value="TETRODE_1.5IN_RADIUS0.25MM"/>
+<part name="16" library="CactusPinInterfaces" deviceset="TETRODE_1.5IN_RADIUS" device="0.25MM" value="TETRODE_1.5IN_RADIUS0.25MM"/>
+<part name="17" library="CactusPinInterfaces" deviceset="TETRODE_1.5IN_RADIUS" device="0.25MM" value="TETRODE_1.5IN_RADIUS0.25MM"/>
+<part name="18" library="CactusPinInterfaces" deviceset="TETRODE_1.5IN_RADIUS" device="0.25MM" value="TETRODE_1.5IN_RADIUS0.25MM"/>
+<part name="19" library="CactusPinInterfaces" deviceset="TETRODE_1.5IN_RADIUS" device="0.25MM" value="TETRODE_1.5IN_RADIUS0.25MM"/>
+<part name="20" library="CactusPinInterfaces" deviceset="TETRODE_1.5IN_RADIUS" device="0.25MM" value="TETRODE_1.5IN_RADIUS0.25MM"/>
+<part name="21" library="CactusPinInterfaces" deviceset="TETRODE_1.5IN_RADIUS" device="0.25MM" value="TETRODE_1.5IN_RADIUS0.25MM"/>
+<part name="22" library="CactusPinInterfaces" deviceset="TETRODE_1.5IN_RADIUS" device="0.25MM" value="TETRODE_1.5IN_RADIUS0.25MM"/>
+<part name="23" library="CactusPinInterfaces" deviceset="TETRODE_1.5IN_RADIUS" device="0.25MM" value="TETRODE_1.5IN_RADIUS0.25MM"/>
+<part name="24" library="CactusPinInterfaces" deviceset="TETRODE_1.5IN_RADIUS" device="0.25MM" value="TETRODE_1.5IN_RADIUS0.25MM"/>
+<part name="25" library="CactusPinInterfaces" deviceset="TETRODE_1.5IN_RADIUS" device="0.25MM" value="TETRODE_1.5IN_RADIUS0.25MM"/>
+<part name="26" library="CactusPinInterfaces" deviceset="TETRODE_1.5IN_RADIUS" device="0.25MM" value="TETRODE_1.5IN_RADIUS0.25MM"/>
+<part name="27" library="CactusPinInterfaces" deviceset="TETRODE_1.5IN_RADIUS" device="0.25MM" value="TETRODE_1.5IN_RADIUS0.25MM"/>
+<part name="28" library="CactusPinInterfaces" deviceset="TETRODE_1.5IN_RADIUS" device="0.25MM" value="TETRODE_1.5IN_RADIUS0.25MM"/>
+<part name="29" library="CactusPinInterfaces" deviceset="TETRODE_1.5IN_RADIUS" device="0.25MM" value="TETRODE_1.5IN_RADIUS0.25MM"/>
+<part name="30" library="CactusPinInterfaces" deviceset="TETRODE_1.5IN_RADIUS" device="0.25MM" value="TETRODE_1.5IN_RADIUS0.25MM"/>
+<part name="31" library="CactusPinInterfaces" deviceset="TETRODE_1.5IN_RADIUS" device="0.25MM" value="TETRODE_1.5IN_RADIUS0.25MM"/>
 </parts>
 <sheets>
