File: OpenEphysHeadstages/RHD2132-Millmax-RightAngle.brd (EAGLE design)
At the start: 22.4 x 26.1 mm, 16 parts, among them U1 RHD2132_QFN

Commit message: Updated solder paste to be little squares for center pads.
Parts:
- S2: device RHD2000:MILLMAX-12PIN-NICE -> RHD2132-Millmax-RightAngle:MILLMAX-12PIN-NICE
- U$1: device voigts:ADXL335 -> RHD2132-Millmax-RightAngle:ADXL335
